Commit message: Add files via upload

File: description/ros2_control.xacro (robot description, xacro)
@@ -5,11 +5,9 @@
         <ros2_control name="RealHardware" type="system">
             <hardware>
-                <plugin>pkg/driver</plugin>
+                <plugin>ros2_control_rover_hardware/RoverHardware</plugin>
                 <!-- Wheel joint names for hardware interface.
                      The *_void_name parameters may be used for slave wheels. -->
                 <param name="left_wheel_name">Fleft_wheel_joint</param>
-                <param name="right_wheel_name">Rright_wheel_joint</param>
-                <param name="left_wheel_void_name">Rleft_wheel_joint</param>
-                <param name="right_wheel_void_name">Fright_wheel_joint</param>
+                <param name="right_wheel_name">Fright_wheel_joint</param>
                 <!-- Encoder counts per revolution for each wheel -->
                 <param name="left_enc_counts_per_rev">2096</param>
@@ -17,6 +15,6 @@
                 <!-- Hardware communication parameters -->
                 <param name="loop_rate">30</param>         <!-- Loop rate in Hz? -->
-                <param name="device">/dev/ttyUSB0</param>  <!-- Serial device -->
-                <param name="baudrate">115200</param>      <!-- Baud rate for serial communication -->
+                <param name="device">/dev/serial/by-id/usb-Silicon_Labs_CP2102_USB_to_UART_Bridge_Controller_0001-if00-port0</param>  <!-- Serial device -->
+                <param name="baud_rate">115200</param>      <!-- Baud rate for serial communication -->
                 <param name="timeout_ms">1000</param>      <!-- Communication timeout in milliseconds -->
             </hardware>
@@ -29,14 +27,6 @@
                     <param name="max">8.7</param>          <!-- Maximum velocity (rad/s) -->
                 </command_interface>
+                <state_interface name="position"/>
                 <state_interface name="velocity"/>
-                <state_interface name="position"/>
-            </joint>
-            <joint name="Rleft_wheel_joint">
-                <command_interface name="velocity">
-                    <param name="min">-8.7</param>
-                    <param name="max">8.7</param>
-                </command_interface>
-                <state_interface name="velocity"/>
-                <state_interface name="position"/>
             </joint>
             <joint name="Fright_wheel_joint">
@@ -45,14 +35,6 @@
                     <param name="max">8.7</param>
                 </command_interface>
+                <state_interface name="position"/>
                 <state_interface name="velocity"/>
-                <state_interface name="position"/>
-            </joint>
-            <joint name="Rright_wheel_joint">
-                <command_interface name="velocity">
-                    <param name="min">-8.7</param>
-                    <param name="max">8.7</param>
-                </command_interface>
-                <state_interface name="velocity"/>
-                <state_interface name="position"/>
             </joint>
         </ros2_control>
